Commit message: Add files via upload

File: rosbot_description/urdf/rosbot.xacro (robot description, xacro)
@@ -256,9 +256,10 @@
   </transmission>
   <!-- Orbbec Astra RGBD Camera -->
-  <joint name="astra_joint" type="fixed">
-    <axis xyz="0 0 0" />
+  <joint name="astra_joint" type="continuous">
     <origin xyz="-0.03 0 0.18" rpy="0 0 0"/>
     <parent link="body_link"/>
     <child link="camera_link"/>
+    <axis xyz="0 0 1"/>
+    <limit effort="25" velocity="1.0" />
   </joint>
   <link name="camera_link">
@@ -277,6 +278,6 @@
     </visual>
     <inertial>
-      <mass value="1e-5" />
-      <origin xyz="0 0 0" rpy="0 0 0"/>
+      <mass value="0.170" />
+      <origin xyz="0 0 0" />
       <inertia ixx="0" ixy="0" ixz="0" iyy="0" iyz="0" izz="0" />
     </inertial>
